Commit message: add left wheel

File: udacity_bot/urdf/udacity_bot.xacro (robot description, xacro)
@@ -55,3 +55,27 @@
     </visual>
   </link>
+  <link name='left_wheel'>
+    <pose>0 0 0 0 1.5707 1.5707</pose>
+    <inertial>
+      <mass value="5.0"/>
+      <origin xyz="0.0 0 0" rpy=" 0 0 0"/>
+      <inertia
+          ixx="0.1" ixy="0" ixz="0"
+          iyy="0.1" iyz="0"
+          izz="0.1"
+      />
+    </inertial>
+    <collision name='collision'>
+      <origin xyz="0 0 0" rpy=" 0 0 0"/>
+      <geometry>
+        <cylinder radius="0.1", length="0.05"/>
+      </geometry>
+    </collision>
+    <visual name='chassis_visual'>
+      <origin xyz="0 0 0" rpy=" 0 0 0"/>
+      <geometry>
+        <cylinder radius="0.1", length="0.05"/>
+      </geometry>
+    </visual>
+  </link>
 </robot>

Commit message: add right wheel

File: udacity_bot/urdf/udacity_bot.xacro (robot description, xacro)
@@ -66,5 +66,5 @@
       />
     </inertial>
-    <collision name='collision'>
+    <collision name='left_wheel_collision'>
       <origin xyz="0 0 0" rpy=" 0 0 0"/>
       <geometry>
@@ -72,5 +72,29 @@
       </geometry>
     </collision>
-    <visual name='chassis_visual'>
+    <visual name='left_wheel_visual'>
+      <origin xyz="0 0 0" rpy=" 0 0 0"/>
+      <geometry>
+        <cylinder radius="0.1", length="0.05"/>
+      </geometry>
+    </visual>
+  </link>
+  <link name='right_wheel'>
+    <pose>0 0 0 0 1.5707 1.5707</pose>
+    <inertial>
+      <mass value="5.0"/>
+      <origin xyz="0.0 0 0" rpy=" 0 0 0"/>
+      <inertia
+          ixx="0.1" ixy="0" ixz="0"
+          iyy="0.1" iyz="0"
+          izz="0.1"
+      />
+    </inertial>
+    <collision name='right_wheel_collision'>
+      <origin xyz="0 0 0" rpy=" 0 0 0"/>
+      <geometry>
+        <cylinder radius="0.1", length="0.05"/>
+      </geometry>
+    </collision>
+    <visual name='right_wheel_visual'>
       <origin xyz="0 0 0" rpy=" 0 0 0"/>
       <geometry>

Commit message: add both wheel hinges

File: udacity_bot/urdf/udacity_bot.xacro (robot description, xacro)
@@ -55,4 +55,12 @@
     </visual>
   </link>
+  <joint type="continuous" name="left_wheel_hinge">
+      <origin xyz="0 0.15 0" rpy="0 0 0"/>
+      <child link="left_wheel"/>
+      <parent link="chassis"/>
+      <axis xyz="0 1 0" rpy="0 0 0"/>
+      <limit effort="10000" velocity="1000"/>
+      <dynamics damping="1.0" friction="1.0"/>
+    </joint>
   <link name='left_wheel'>
     <pose>0 0 0 0 1.5707 1.5707</pose>
@@ -79,4 +87,12 @@
     </visual>
   </link>
+  <joint type="continuous" name="right_wheel_hinge">
+      <origin xyz="0 -0.15 0" rpy="0 0 0"/>
+      <child link="left_wheel"/>
+      <parent link="chassis"/>
+      <axis xyz="0 1 0" rpy="0 0 0"/>
+      <limit effort="10000" velocity="1000"/>
+      <dynamics damping="1.0" friction="1.0"/>
+    </joint>
   <link name='right_wheel'>
     <pose>0 0 0 0 1.5707 1.5707</pose>

Commit message: wrong format. no comma

File: udacity_bot/urdf/udacity_bot.xacro (robot description, xacro)
@@ -77,5 +77,5 @@
       <origin xyz="0 0 0" rpy=" 0 0 0"/>
       <geometry>
-        <cylinder radius="0.1", length="0.05"/>
+        <cylinder radius="0.1" length="0.05"/>
       </geometry>
     </collision>
@@ -83,5 +83,5 @@
       <origin xyz="0 0 0" rpy=" 0 0 0"/>
       <geometry>
-        <cylinder radius="0.1", length="0.05"/>
+        <cylinder radius="0.1" length="0.05"/>
       </geometry>
     </visual>
@@ -109,5 +109,5 @@
       <origin xyz="0 0 0" rpy=" 0 0 0"/>
       <geometry>
-        <cylinder radius="0.1", length="0.05"/>
+        <cylinder radius="0.1" length="0.05"/>
       </geometry>
     </collision>
@@ -115,5 +115,5 @@
       <origin xyz="0 0 0" rpy=" 0 0 0"/>
       <geometry>
-        <cylinder radius="0.1", length="0.05"/>
+        <cylinder radius="0.1" length="0.05"/>
       </geometry>
     </visual>

Commit message: wrong format. no comma

File: udacity_bot/urdf/udacity_bot.xacro (robot description, xacro)
@@ -77,5 +77,5 @@
       <origin xyz="0 0 0" rpy=" 0 0 0"/>
       <geometry>
-        <cylinder radius="0.1", length="0.05"/>
+        <cylinder radius="0.1" length="0.05"/>
       </geometry>
     </collision>
@@ -83,5 +83,5 @@
       <origin xyz="0 0 0" rpy=" 0 0 0"/>
       <geometry>
-        <cylinder radius="0.1", length="0.05"/>
+        <cylinder radius="0.1" length="0.05"/>
       </geometry>
     </visual>

Commit message: wrong link for the right wheel hinge

File: udacity_bot/urdf/udacity_bot.xacro (robot description, xacro)
@@ -89,5 +89,5 @@
   <joint type="continuous" name="right_wheel_hinge">
       <origin xyz="0 -0.15 0" rpy="0 0 0"/>
-      <child link="left_wheel"/>
+      <child link="right_wheel"/>
       <parent link="chassis"/>
       <axis xyz="0 1 0" rpy="0 0 0"/>

Commit message: axis might be wrong, try z

File: udacity_bot/urdf/udacity_bot.xacro (robot description, xacro)
@@ -59,5 +59,5 @@
       <child link="left_wheel"/>
       <parent link="chassis"/>
-      <axis xyz="0 1 0" rpy="0 0 0"/>
+      <axis xyz="0 0 1" rpy="0 0 0"/>
       <limit effort="10000" velocity="1000"/>
       <dynamics damping="1.0" friction="1.0"/>
@@ -91,5 +91,5 @@
       <child link="right_wheel"/>
       <parent link="chassis"/>
-      <axis xyz="0 1 0" rpy="0 0 0"/>
+      <axis xyz="0 0 1" rpy="0 0 0"/>
       <limit effort="10000" velocity="1000"/>
       <dynamics damping="1.0" friction="1.0"/>

Commit message: Revert "axis might be wrong, try z"
This reverts commit c6b7797e7ef62330dfcffcba28b377bf397216cf.

File: udacity_bot/urdf/udacity_bot.xacro (robot description, xacro)
@@ -59,5 +59,5 @@
       <child link="left_wheel"/>
       <parent link="chassis"/>
-      <axis xyz="0 0 1" rpy="0 0 0"/>
+      <axis xyz="0 1 0" rpy="0 0 0"/>
       <limit effort="10000" velocity="1000"/>
       <dynamics damping="1.0" friction="1.0"/>
@@ -91,5 +91,5 @@
       <child link="right_wheel"/>
       <parent link="chassis"/>
-      <axis xyz="0 0 1" rpy="0 0 0"/>
+      <axis xyz="0 1 0" rpy="0 0 0"/>
       <limit effort="10000" velocity="1000"/>
       <dynamics damping="1.0" friction="1.0"/>

Commit message: should have used this attribute
and all three of them inside each category should be the same

File: udacity_bot/urdf/udacity_bot.xacro (robot description, xacro)
@@ -66,5 +66,5 @@
     <inertial>
       <mass value="5.0"/>
-      <origin xyz="0.0 0 0" rpy=" 0 0 0"/>
+      <origin xyz="0.0 0 0" rpy=" 0 1.5707 1.5707"/>
       <inertia
           ixx="0.1" ixy="0" ixz="0"
@@ -74,5 +74,5 @@
     </inertial>
     <collision name='left_wheel_collision'>
-      <origin xyz="0 0 0" rpy=" 0 0 0"/>
+      <origin xyz="0.0 0 0" rpy=" 0 1.5707 1.5707"/>
       <geometry>
         <cylinder radius="0.1" length="0.05"/>
@@ -80,5 +80,5 @@
     </collision>
     <visual name='left_wheel_visual'>
-      <origin xyz="0 0 0" rpy=" 0 0 0"/>
+      <origin xyz="0.0 0 0" rpy=" 0 1.5707 1.5707"/>
       <geometry>
         <cylinder radius="0.1" length="0.05"/>
@@ -97,5 +97,5 @@
     <inertial>
       <mass value="5.0"/>
-      <origin xyz="0.0 0 0" rpy=" 0 0 0"/>
+      <origin xyz="0.0 0 0" rpy=" 0 1.5707 1.5707"/>
       <inertia
           ixx="0.1" ixy="0" ixz="0"
@@ -105,5 +105,5 @@
     </inertial>
     <collision name='right_wheel_collision'>
-      <origin xyz="0 0 0" rpy=" 0 0 0"/>
+      <origin xyz="0.0 0 0" rpy=" 0 1.5707 1.5707"/>
       <geometry>
         <cylinder radius="0.1" length="0.05"/>
@@ -111,5 +111,5 @@
     </collision>
     <visual name='right_wheel_visual'>
-      <origin xyz="0 0 0" rpy=" 0 0 0"/>
+      <origin xyz="0.0 0 0" rpy=" 0 1.5707 1.5707"/>
       <geometry>
         <cylinder radius="0.1" length="0.05"/>

Commit message: reformat

File: udacity_bot/urdf/udacity_bot.xacro (robot description, xacro)
@@ -3,7 +3,7 @@
   <link name="robot_footprint"></link>
   <joint name="robot_footprint_joint" type="fixed">
-    <origin xyz="0 0 0" rpy="0 0 0" />
+    <origin xyz="0 0 0" rpy="0 0 0"/>
     <parent link="robot_footprint"/>
-    <child link="chassis" />
+    <child link="chassis"/>
   </joint>
   <link name='chassis'>
@@ -12,9 +12,5 @@
       <mass value="15.0"/>
       <origin xyz="0.0 0 0" rpy=" 0 0 0"/>
-      <inertia
-          ixx="0.1" ixy="0" ixz="0"
-          iyy="0.1" iyz="0"
-          izz="0.1"
-      />
+      <inertia ixx="0.1" ixy="0" ixz="0" iyy="0.1" iyz="0" izz="0.1"/>
     </inertial>
     <collision name='collision'>
@@ -56,20 +52,16 @@
   </link>
   <joint type="continuous" name="left_wheel_hinge">
-      <origin xyz="0 0.15 0" rpy="0 0 0"/>
-      <child link="left_wheel"/>
-      <parent link="chassis"/>
-      <axis xyz="0 1 0" rpy="0 0 0"/>
-      <limit effort="10000" velocity="1000"/>
-      <dynamics damping="1.0" friction="1.0"/>
-    </joint>
+    <origin xyz="0 0.15 0" rpy="0 0 0"/>
+    <child link="left_wheel"/>
+    <parent link="chassis"/>
+    <axis xyz="0 1 0" rpy="0 0 0"/>
+    <limit effort="10000" velocity="1000"/>
+    <dynamics damping="1.0" friction="1.0"/>
+  </joint>
   <link name='left_wheel'>
     <inertial>
       <mass value="5.0"/>
       <origin xyz="0.0 0 0" rpy=" 0 1.5707 1.5707"/>
-      <inertia
-          ixx="0.1" ixy="0" ixz="0"
-          iyy="0.1" iyz="0"
-          izz="0.1"
-      />
+      <inertia ixx="0.1" ixy="0" ixz="0" iyy="0.1" iyz="0" izz="0.1"/>
     </inertial>
     <collision name='left_wheel_collision'>
@@ -87,20 +79,16 @@
   </link>
   <joint type="continuous" name="right_wheel_hinge">
-      <origin xyz="0 -0.15 0" rpy="0 0 0"/>
-      <child link="right_wheel"/>
-      <parent link="chassis"/>
-      <axis xyz="0 1 0" rpy="0 0 0"/>
-      <limit effort="10000" velocity="1000"/>
-      <dynamics damping="1.0" friction="1.0"/>
-    </joint>
+    <origin xyz="0 -0.15 0" rpy="0 0 0"/>
+    <child link="right_wheel"/>
+    <parent link="chassis"/>
+    <axis xyz="0 1 0" rpy="0 0 0"/>
+    <limit effort="10000" velocity="1000"/>
+    <dynamics damping="1.0" friction="1.0"/>
+  </joint>
   <link name='right_wheel'>
     <inertial>
       <mass value="5.0"/>
       <origin xyz="0.0 0 0" rpy=" 0 1.5707 1.5707"/>
-      <inertia
-          ixx="0.1" ixy="0" ixz="0"
-          iyy="0.1" iyz="0"
-          izz="0.1"
-      />
+      <inertia ixx="0.1" ixy="0" ixz="0" iyy="0.1" iyz="0" izz="0.1"/>
     </inertial>
     <collision name='right_wheel_collision'>

Commit message: add camera link and joint

File: udacity_bot/urdf/udacity_bot.xacro (robot description, xacro)
@@ -105,3 +105,27 @@
     </visual>
   </link>
+  <link name='camera'>
+    <inertial>
+      <mass value="0.1"/>
+      <origin xyz="0.0 0 0" rpy=" 0 0 0"/>
+      <inertia ixx="1e-6" ixy="0" ixz="0" iyy="1e-6" iyz="0" izz="1e-6"/>
+    </inertial>
+    <collision name='camera_collision'>
+      <origin xyz="0.0 0 0" rpy=" 0 0 0"/>
+      <geometry>
+        <box size=".05 .05 .05"/>
+      </geometry>
+    </collision>
+    <visual name='camera_visual'>
+      <origin xyz="0.0 0 0" rpy=" 0 0 0"/>
+      <geometry>
+        <box size=".05 .05 .05"/>
+      </geometry>
+    </visual>
+  </link>
+  <joint type="fixed" name="camera_joint">
+    <origin xyz="0.2 0 0" rpy="0 0 0"/>
+    <child link="camera"/>
+    <parent link="chassis"/>
+  </joint>
 </robot>

Commit message: add laser range finder

File: udacity_bot/urdf/udacity_bot.xacro (robot description, xacro)
@@ -129,3 +129,27 @@
     <parent link="chassis"/>
   </joint>
+  <link name='hokuyo'>
+    <inertial>
+      <mass value="0.1"/>
+      <origin xyz="0.0 0 0" rpy=" 0 0 0"/>
+      <inertia ixx="1e-6" ixy="0" ixz="0" iyy="1e-6" iyz="0" izz="1e-6"/>
+    </inertial>
+    <collision name='hokuyo_collision'>
+      <origin xyz="0.0 0 0" rpy=" 0 0 0"/>
+      <geometry>
+        <box size=".1 .1 .1"/>
+      </geometry>
+    </collision>
+    <visual name='hokuyo_visual'>
+      <origin xyz="0.0 0 0" rpy=" 0 0 0"/>
+      <geometry>
+        <mesh filename="package://udacity_bot/meshes/hokuyo.dae"/>
+      </geometry>
+    </visual>
+  </link>
+  <joint type="fixed" name="hokuyo_joint">
+    <origin xyz=".15 0 .1" rpy="0 0 0"/>
+    <child link="hokuyo"/>
+    <parent link="chassis"/>
+  </joint>
 </robot>
