Commit message: adjust the sizes of the parts

File: roborock/urdf/roborock.xacro (robot description, xacro)
@@ -18,5 +18,5 @@
       <origin xyz="0 0 0" rpy=" 0 0 0"/>
       <geometry>
-        <cylinder radius="0.8" length="0.1"/>
+        <cylinder radius="0.5" length="0.1"/>
       </geometry>
     </collision>
@@ -24,5 +24,5 @@
       <origin xyz="0 0 0" rpy=" 0 0 0"/>
       <geometry>
-        <cylinder radius="0.8" length="0.1"/>
+        <cylinder radius="0.5" length="0.1"/>
       </geometry>
     </visual>
@@ -69,5 +69,5 @@
       <origin xyz="0.0 0 0" rpy=" 0 1.5707 1.5707"/>
       <geometry>
-        <cylinder radius="0.05" length="0.05"/>
+        <cylinder radius="0.08" length="0.05"/>
       </geometry>
     </collision>
@@ -75,5 +75,5 @@
       <origin xyz="0.0 0 0" rpy=" 0 1.5707 1.5707"/>
       <geometry>
-        <cylinder radius="0.05" length="0.05"/>
+        <cylinder radius="0.08" length="0.05"/>
       </geometry>
     </visual>
@@ -96,5 +96,5 @@
       <origin xyz="0.0 0 0" rpy=" 0 1.5707 1.5707"/>
       <geometry>
-        <cylinder radius="0.05" length="0.05"/>
+        <cylinder radius="0.08" length="0.05"/>
       </geometry>
     </collision>
@@ -102,5 +102,5 @@
       <origin xyz="0.0 0 0" rpy=" 0 1.5707 1.5707"/>
       <geometry>
-        <cylinder radius="0.05" length="0.05"/>
+        <cylinder radius="0.08" length="0.05"/>
       </geometry>
     </visual>

Commit message: replace the package names

File: roborock/urdf/roborock.xacro (robot description, xacro)
@@ -145,5 +145,5 @@
       <origin xyz="0.0 0 0" rpy=" 0 0 0"/>
       <geometry>
-        <mesh filename="package://udacity_bot/meshes/hokuyo.dae"/>
+        <mesh filename="package://roborock/meshes/hokuyo.dae"/>
       </geometry>
     </visual>

Commit message: adjust the parts

File: roborock/urdf/roborock.xacro (robot description, xacro)
@@ -18,5 +18,5 @@
       <origin xyz="0 0 0" rpy=" 0 0 0"/>
       <geometry>
-        <cylinder radius="0.5" length="0.1"/>
+        <cylinder radius="0.4" length="0.1"/>
       </geometry>
     </collision>
@@ -24,5 +24,5 @@
       <origin xyz="0 0 0" rpy=" 0 0 0"/>
       <geometry>
-        <cylinder radius="0.5" length="0.1"/>
+        <cylinder radius="0.4" length="0.1"/>
       </geometry>
     </visual>
@@ -53,5 +53,5 @@
   </link>
   <joint type="continuous" name="left_wheel_hinge">
-    <origin xyz="0 0.15 0" rpy="0 0 0"/>
+    <origin xyz="0 0.25 -0.05" rpy="0 0 0"/>
     <child link="left_wheel"/>
     <parent link="chassis"/>
@@ -69,5 +69,5 @@
       <origin xyz="0.0 0 0" rpy=" 0 1.5707 1.5707"/>
       <geometry>
-        <cylinder radius="0.08" length="0.05"/>
+        <cylinder radius="0.1" length="0.05"/>
       </geometry>
     </collision>
@@ -75,10 +75,10 @@
       <origin xyz="0.0 0 0" rpy=" 0 1.5707 1.5707"/>
       <geometry>
-        <cylinder radius="0.08" length="0.05"/>
+        <cylinder radius="0.1" length="0.05"/>
       </geometry>
     </visual>
   </link>
   <joint type="continuous" name="right_wheel_hinge">
-    <origin xyz="0 -0.15 0" rpy="0 0 0"/>
+    <origin xyz="0 -0.25 -0.05" rpy="0 0 0"/>
     <child link="right_wheel"/>
     <parent link="chassis"/>
@@ -96,5 +96,5 @@
       <origin xyz="0.0 0 0" rpy=" 0 1.5707 1.5707"/>
       <geometry>
-        <cylinder radius="0.08" length="0.05"/>
+        <cylinder radius="0.1" length="0.05"/>
       </geometry>
     </collision>
@@ -102,5 +102,5 @@
       <origin xyz="0.0 0 0" rpy=" 0 1.5707 1.5707"/>
       <geometry>
-        <cylinder radius="0.08" length="0.05"/>
+        <cylinder radius="0.1" length="0.05"/>
       </geometry>
     </visual>
@@ -126,5 +126,5 @@
   </link>
   <joint type="fixed" name="camera_joint">
-    <origin xyz="0.2 0 0" rpy="0 0 0"/>
+    <origin xyz="0.45 0 0" rpy="0 0 0"/>
     <child link="camera"/>
     <parent link="chassis"/>
@@ -150,5 +150,5 @@
   </link>
   <joint type="fixed" name="hokuyo_joint">
-    <origin xyz="-0.15 0 .1" rpy="0 0 0"/>
+    <origin xyz="-0.2 0 .1" rpy="0 0 0"/>
     <child link="hokuyo"/>
     <parent link="chassis"/>

Commit message: lower the caster

File: roborock/urdf/roborock.xacro (robot description, xacro)
@@ -28,5 +28,5 @@
     </visual>
     <collision name='back_caster_collision'>
-      <origin xyz="-0.15 0 -0.05" rpy=" 0 0 0"/>
+      <origin xyz="-0.15 0 -0.1" rpy=" 0 0 0"/>
       <geometry>
         <sphere radius="0.0499"/>
@@ -34,5 +34,5 @@
     </collision>
     <visual name='back_caster_visual'>
-      <origin xyz="-0.15 0 -0.05" rpy=" 0 0 0"/>
+      <origin xyz="-0.15 0 -0.1" rpy=" 0 0 0"/>
       <geometry>
         <sphere radius="0.05"/>
@@ -40,5 +40,5 @@
     </visual>
     <collision name='front_caster_collision'>
-      <origin xyz="0.15 0 -0.05" rpy=" 0 0 0"/>
+      <origin xyz="0.15 0 -0.1" rpy=" 0 0 0"/>
       <geometry>
         <sphere radius="0.0499"/>
@@ -46,5 +46,5 @@
     </collision>
     <visual name='front_caster_visual'>
-      <origin xyz="0.15 0 -0.05" rpy=" 0 0 0"/>
+      <origin xyz="0.15 0 -0.1" rpy=" 0 0 0"/>
       <geometry>
         <sphere radius="0.05"/>

Commit message: make the chassis thicker

File: roborock/urdf/roborock.xacro (robot description, xacro)
@@ -18,5 +18,5 @@
       <origin xyz="0 0 0" rpy=" 0 0 0"/>
       <geometry>
-        <cylinder radius="0.4" length="0.1"/>
+        <cylinder radius="0.4" length="0.15"/>
       </geometry>
     </collision>
@@ -24,5 +24,5 @@
       <origin xyz="0 0 0" rpy=" 0 0 0"/>
       <geometry>
-        <cylinder radius="0.4" length="0.1"/>
+        <cylinder radius="0.4" length="0.15"/>
       </geometry>
     </visual>

Commit message: raise the hinges and casters

File: roborock/urdf/roborock.xacro (robot description, xacro)
@@ -28,5 +28,5 @@
     </visual>
     <collision name='back_caster_collision'>
-      <origin xyz="-0.15 0 -0.1" rpy=" 0 0 0"/>
+      <origin xyz="-0.25 0 -0.05" rpy=" 0 0 0"/>
       <geometry>
         <sphere radius="0.0499"/>
@@ -34,5 +34,5 @@
     </collision>
     <visual name='back_caster_visual'>
-      <origin xyz="-0.15 0 -0.1" rpy=" 0 0 0"/>
+      <origin xyz="-0.25 0 -0.05" rpy=" 0 0 0"/>
       <geometry>
         <sphere radius="0.05"/>
@@ -40,5 +40,5 @@
     </visual>
     <collision name='front_caster_collision'>
-      <origin xyz="0.15 0 -0.1" rpy=" 0 0 0"/>
+      <origin xyz="0.25 0 -0.05" rpy=" 0 0 0"/>
       <geometry>
         <sphere radius="0.0499"/>
@@ -46,5 +46,5 @@
     </collision>
     <visual name='front_caster_visual'>
-      <origin xyz="0.15 0 -0.1" rpy=" 0 0 0"/>
+      <origin xyz="0.25 0 -0.05" rpy=" 0 0 0"/>
       <geometry>
         <sphere radius="0.05"/>
@@ -53,5 +53,5 @@
   </link>
   <joint type="continuous" name="left_wheel_hinge">
-    <origin xyz="0 0.25 -0.05" rpy="0 0 0"/>
+    <origin xyz="0 0.25 0" rpy="0 0 0"/>
     <child link="left_wheel"/>
     <parent link="chassis"/>
@@ -80,5 +80,5 @@
   </link>
   <joint type="continuous" name="right_wheel_hinge">
-    <origin xyz="0 -0.25 -0.05" rpy="0 0 0"/>
+    <origin xyz="0 -0.25 0" rpy="0 0 0"/>
     <child link="right_wheel"/>
     <parent link="chassis"/>

Commit message: lower the hinge and casters so they stay inside

File: roborock/urdf/roborock.xacro (robot description, xacro)
@@ -28,5 +28,5 @@
     </visual>
     <collision name='back_caster_collision'>
-      <origin xyz="-0.25 0 -0.05" rpy=" 0 0 0"/>
+      <origin xyz="-0.25 0 -0.075" rpy=" 0 0 0"/>
       <geometry>
         <sphere radius="0.0499"/>
@@ -34,5 +34,5 @@
     </collision>
     <visual name='back_caster_visual'>
-      <origin xyz="-0.25 0 -0.05" rpy=" 0 0 0"/>
+      <origin xyz="-0.25 0 -0.075" rpy=" 0 0 0"/>
       <geometry>
         <sphere radius="0.05"/>
@@ -40,5 +40,5 @@
     </visual>
     <collision name='front_caster_collision'>
-      <origin xyz="0.25 0 -0.05" rpy=" 0 0 0"/>
+      <origin xyz="0.25 0 -0.075" rpy=" 0 0 0"/>
       <geometry>
         <sphere radius="0.0499"/>
@@ -46,5 +46,5 @@
     </collision>
     <visual name='front_caster_visual'>
-      <origin xyz="0.25 0 -0.05" rpy=" 0 0 0"/>
+      <origin xyz="0.25 0 -0.075" rpy=" 0 0 0"/>
       <geometry>
         <sphere radius="0.05"/>
@@ -53,5 +53,5 @@
   </link>
   <joint type="continuous" name="left_wheel_hinge">
-    <origin xyz="0 0.25 0" rpy="0 0 0"/>
+    <origin xyz="0 0.25 -0.025" rpy="0 0 0"/>
     <child link="left_wheel"/>
     <parent link="chassis"/>
@@ -80,5 +80,5 @@
   </link>
   <joint type="continuous" name="right_wheel_hinge">
-    <origin xyz="0 -0.25 0" rpy="0 0 0"/>
+    <origin xyz="0 -0.25 -0.025" rpy="0 0 0"/>
     <child link="right_wheel"/>
     <parent link="chassis"/>
@@ -126,5 +126,5 @@
   </link>
   <joint type="fixed" name="camera_joint">
-    <origin xyz="0.45 0 0" rpy="0 0 0"/>
+    <origin xyz="0.4 0 0" rpy="0 0 0"/>
     <child link="camera"/>
     <parent link="chassis"/>

Commit message: add materials

File: roborock/urdf/roborock.xacro (robot description, xacro)
@@ -2,4 +2,10 @@
 <robot name="roborock" xmlns:xacro="http://www.ros.org/wiki/xacro">
   <xacro:include filename="$(find roborock)/urdf/roborock.gazebo"/>
+  <material name="army_green">
+    <color rgba="45 134 45 1"/>
+    </material>
+  <material name="black">
+    <color rgba="0 0 0 1"/>
+  </material>
   <link name="robot_footprint"></link>
   <joint name="robot_footprint_joint" type="fixed">
@@ -26,4 +32,5 @@
         <cylinder radius="0.4" length="0.15"/>
       </geometry>
+      <material name="army_green">
     </visual>
     <collision name='back_caster_collision'>
@@ -77,4 +84,5 @@
         <cylinder radius="0.1" length="0.05"/>
       </geometry>
+      <material name="black">
     </visual>
   </link>
@@ -104,4 +112,5 @@
         <cylinder radius="0.1" length="0.05"/>
       </geometry>
+      <material name="black">
     </visual>
   </link>

Commit message: wrong format

File: roborock/urdf/roborock.xacro (robot description, xacro)
@@ -32,5 +32,5 @@
         <cylinder radius="0.4" length="0.15"/>
       </geometry>
-      <material name="army_green">
+      <material name="army_green" />
     </visual>
     <collision name='back_caster_collision'>
@@ -84,5 +84,5 @@
         <cylinder radius="0.1" length="0.05"/>
       </geometry>
-      <material name="black">
+      <material name="black"/>
     </visual>
   </link>
@@ -112,5 +112,5 @@
         <cylinder radius="0.1" length="0.05"/>
       </geometry>
-      <material name="black">
+      <material name="black"/>
     </visual>
   </link>

Commit message: reformat

File: roborock/urdf/roborock.xacro (robot description, xacro)
@@ -1,165 +1,165 @@
 <?xml version='1.0'?>
 <robot name="roborock" xmlns:xacro="http://www.ros.org/wiki/xacro">
-  <xacro:include filename="$(find roborock)/urdf/roborock.gazebo"/>
-  <material name="army_green">
-    <color rgba="45 134 45 1"/>
+    <xacro:include filename="$(find roborock)/urdf/roborock.gazebo"/>
+    <material name="army_green">
+        <color rgba="45 134 45 1"/>
     </material>
-  <material name="black">
-    <color rgba="0 0 0 1"/>
-  </material>
-  <link name="robot_footprint"></link>
-  <joint name="robot_footprint_joint" type="fixed">
-    <origin xyz="0 0 0" rpy="0 0 0"/>
-    <parent link="robot_footprint"/>
-    <child link="chassis"/>
-  </joint>
-  <link name='chassis'>
-    <pose>0 0 0.1 0 0 0</pose>
-    <inertial>
-      <mass value="15.0"/>
-      <origin xyz="0.0 0 0" rpy=" 0 0 0"/>
-      <inertia ixx="0.1" ixy="0" ixz="0" iyy="0.1" iyz="0" izz="0.1"/>
-    </inertial>
-    <collision name='collision'>
-      <origin xyz="0 0 0" rpy=" 0 0 0"/>
-      <geometry>
-        <cylinder radius="0.4" length="0.15"/>
-      </geometry>
-    </collision>
-    <visual name='chassis_visual'>
-      <origin xyz="0 0 0" rpy=" 0 0 0"/>
-      <geometry>
-        <cylinder radius="0.4" length="0.15"/>
-      </geometry>
-      <material name="army_green" />
-    </visual>
-    <collision name='back_caster_collision'>
-      <origin xyz="-0.25 0 -0.075" rpy=" 0 0 0"/>
-      <geometry>
-        <sphere radius="0.0499"/>
-      </geometry>
-    </collision>
-    <visual name='back_caster_visual'>
-      <origin xyz="-0.25 0 -0.075" rpy=" 0 0 0"/>
-      <geometry>
-        <sphere radius="0.05"/>
-      </geometry>
-    </visual>
-    <collision name='front_caster_collision'>
-      <origin xyz="0.25 0 -0.075" rpy=" 0 0 0"/>
-      <geometry>
-        <sphere radius="0.0499"/>
-      </geometry>
-    </collision>
-    <visual name='front_caster_visual'>
-      <origin xyz="0.25 0 -0.075" rpy=" 0 0 0"/>
-      <geometry>
-        <sphere radius="0.05"/>
-      </geometry>
-    </visual>
-  </link>
-  <joint type="continuous" name="left_wheel_hinge">
-    <origin xyz="0 0.25 -0.025" rpy="0 0 0"/>
-    <child link="left_wheel"/>
-    <parent link="chassis"/>
-    <axis xyz="0 1 0" rpy="0 0 0"/>
-    <limit effort="10000" velocity="1000"/>
-    <dynamics damping="1.0" friction="1.0"/>
-  </joint>
-  <link name='left_wheel'>
-    <inertial>
-      <mass value="5.0"/>
-      <origin xyz="0.0 0 0" rpy=" 0 1.5707 1.5707"/>
-      <inertia ixx="0.1" ixy="0" ixz="0" iyy="0.1" iyz="0" izz="0.1"/>
-    </inertial>
-    <collision name='left_wheel_collision'>
-      <origin xyz="0.0 0 0" rpy=" 0 1.5707 1.5707"/>
-      <geometry>
-        <cylinder radius="0.1" length="0.05"/>
-      </geometry>
-    </collision>
-    <visual name='left_wheel_visual'>
-      <origin xyz="0.0 0 0" rpy=" 0 1.5707 1.5707"/>
-      <geometry>
-        <cylinder radius="0.1" length="0.05"/>
-      </geometry>
-      <material name="black"/>
-    </visual>
-  </link>
-  <joint type="continuous" name="right_wheel_hinge">
-    <origin xyz="0 -0.25 -0.025" rpy="0 0 0"/>
-    <child link="right_wheel"/>
-    <parent link="chassis"/>
-    <axis xyz="0 1 0" rpy="0 0 0"/>
-    <limit effort="10000" velocity="1000"/>
-    <dynamics damping="1.0" friction="1.0"/>
-  </joint>
-  <link name='right_wheel'>
-    <inertial>
-      <mass value="5.0"/>
-      <origin xyz="0.0 0 0" rpy=" 0 1.5707 1.5707"/>
-      <inertia ixx="0.1" ixy="0" ixz="0" iyy="0.1" iyz="0" izz="0.1"/>
-    </inertial>
-    <collision name='right_wheel_collision'>
-      <origin xyz="0.0 0 0" rpy=" 0 1.5707 1.5707"/>
-      <geometry>
-        <cylinder radius="0.1" length="0.05"/>
-      </geometry>
-    </collision>
-    <visual name='right_wheel_visual'>
-      <origin xyz="0.0 0 0" rpy=" 0 1.5707 1.5707"/>
-      <geometry>
-        <cylinder radius="0.1" length="0.05"/>
-      </geometry>
-      <material name="black"/>
-    </visual>
-  </link>
-  <link name='camera'>
-    <inertial>
-      <mass value="0.1"/>
-      <origin xyz="0.0 0 0" rpy=" 0 0 0"/>
-      <inertia ixx="1e-6" ixy="0" ixz="0" iyy="1e-6" iyz="0" izz="1e-6"/>
-    </inertial>
-    <collision name='camera_collision'>
-      <origin xyz="0.0 0 0" rpy=" 0 0 0"/>
-      <geometry>
-        <box size=".05 .05 .05"/>
-      </geometry>
-    </collision>
-    <visual name='camera_visual'>
-      <origin xyz="0.0 0 0" rpy=" 0 0 0"/>
-      <geometry>
-        <box size=".05 .05 .05"/>
-      </geometry>
-    </visual>
-  </link>
-  <joint type="fixed" name="camera_joint">
-    <origin xyz="0.4 0 0" rpy="0 0 0"/>
-    <child link="camera"/>
-    <parent link="chassis"/>
-  </joint>
-  <link name='hokuyo'>
-    <inertial>
-      <mass value="0.1"/>
-      <origin xyz="0.0 0 0" rpy=" 0 0 0"/>
-      <inertia ixx="1e-6" ixy="0" ixz="0" iyy="1e-6" iyz="0" izz="1e-6"/>
-    </inertial>
-    <collision name='hokuyo_collision'>
-      <origin xyz="0.0 0 0" rpy=" 0 0 0"/>
-      <geometry>
-        <box size=".1 .1 .1"/>
-      </geometry>
-    </collision>
-    <visual name='hokuyo_visual'>
-      <origin xyz="0.0 0 0" rpy=" 0 0 0"/>
-      <geometry>
-        <mesh filename="package://roborock/meshes/hokuyo.dae"/>
-      </geometry>
-    </visual>
-  </link>
-  <joint type="fixed" name="hokuyo_joint">
-    <origin xyz="-0.2 0 .1" rpy="0 0 0"/>
-    <child link="hokuyo"/>
-    <parent link="chassis"/>
-  </joint>
+    <material name="black">
+        <color rgba="0 0 0 1"/>
+    </material>
+    <link name="robot_footprint"></link>
+    <joint name="robot_footprint_joint" type="fixed">
+        <origin xyz="0 0 0" rpy="0 0 0"/>
+        <parent link="robot_footprint"/>
+        <child link="chassis"/>
+    </joint>
+    <link name='chassis'>
+        <pose>0 0 0.1 0 0 0</pose>
+        <inertial>
+            <mass value="15.0"/>
+            <origin xyz="0.0 0 0" rpy=" 0 0 0"/>
+            <inertia ixx="0.1" ixy="0" ixz="0" iyy="0.1" iyz="0" izz="0.1"/>
+        </inertial>
+        <collision name='collision'>
+            <origin xyz="0 0 0" rpy=" 0 0 0"/>
+            <geometry>
+                <cylinder radius="0.4" length="0.15"/>
+            </geometry>
+        </collision>
+        <visual name='chassis_visual'>
+            <origin xyz="0 0 0" rpy=" 0 0 0"/>
+            <geometry>
+                <cylinder radius="0.4" length="0.15"/>
+            </geometry>
+            <material name="army_green"/>
+        </visual>
+        <collision name='back_caster_collision'>
+            <origin xyz="-0.25 0 -0.075" rpy=" 0 0 0"/>
+            <geometry>
+                <sphere radius="0.0499"/>
+            </geometry>
+        </collision>
+        <visual name='back_caster_visual'>
+            <origin xyz="-0.25 0 -0.075" rpy=" 0 0 0"/>
+            <geometry>
+                <sphere radius="0.05"/>
+            </geometry>
+        </visual>
+        <collision name='front_caster_collision'>
+            <origin xyz="0.25 0 -0.075" rpy=" 0 0 0"/>
+            <geometry>
+                <sphere radius="0.0499"/>
+            </geometry>
+        </collision>
+        <visual name='front_caster_visual'>
+            <origin xyz="0.25 0 -0.075" rpy=" 0 0 0"/>
+            <geometry>
+                <sphere radius="0.05"/>
+            </geometry>
+        </visual>
+    </link>
+    <joint type="continuous" name="left_wheel_hinge">
+        <origin xyz="0 0.25 -0.025" rpy="0 0 0"/>
+        <child link="left_wheel"/>
+        <parent link="chassis"/>
+        <axis xyz="0 1 0" rpy="0 0 0"/>
+        <limit effort="10000" velocity="1000"/>
+        <dynamics damping="1.0" friction="1.0"/>
+    </joint>
+    <link name='left_wheel'>
+        <inertial>
+            <mass value="5.0"/>
+            <origin xyz="0.0 0 0" rpy=" 0 1.5707 1.5707"/>
+            <inertia ixx="0.1" ixy="0" ixz="0" iyy="0.1" iyz="0" izz="0.1"/>
+        </inertial>
+        <collision name='left_wheel_collision'>
+            <origin xyz="0.0 0 0" rpy=" 0 1.5707 1.5707"/>
+            <geometry>
+                <cylinder radius="0.1" length="0.05"/>
+            </geometry>
+        </collision>
+        <visual name='left_wheel_visual'>
+            <origin xyz="0.0 0 0" rpy=" 0 1.5707 1.5707"/>
+            <geometry>
+                <cylinder radius="0.1" length="0.05"/>
+            </geometry>
+            <material name="black"/>
+        </visual>
+    </link>
+    <joint type="continuous" name="right_wheel_hinge">
+        <origin xyz="0 -0.25 -0.025" rpy="0 0 0"/>
+        <child link="right_wheel"/>
+        <parent link="chassis"/>
+        <axis xyz="0 1 0" rpy="0 0 0"/>
+        <limit effort="10000" velocity="1000"/>
+        <dynamics damping="1.0" friction="1.0"/>
+    </joint>
+    <link name='right_wheel'>
+        <inertial>
+            <mass value="5.0"/>
+            <origin xyz="0.0 0 0" rpy=" 0 1.5707 1.5707"/>
+            <inertia ixx="0.1" ixy="0" ixz="0" iyy="0.1" iyz="0" izz="0.1"/>
+        </inertial>
+        <collision name='right_wheel_collision'>
+            <origin xyz="0.0 0 0" rpy=" 0 1.5707 1.5707"/>
+            <geometry>
+                <cylinder radius="0.1" length="0.05"/>
+            </geometry>
+        </collision>
+        <visual name='right_wheel_visual'>
+            <origin xyz="0.0 0 0" rpy=" 0 1.5707 1.5707"/>
+            <geometry>
+                <cylinder radius="0.1" length="0.05"/>
+            </geometry>
+            <material name="black"/>
+        </visual>
+    </link>
+    <link name='camera'>
+        <inertial>
+            <mass value="0.1"/>
+            <origin xyz="0.0 0 0" rpy=" 0 0 0"/>
+            <inertia ixx="1e-6" ixy="0" ixz="0" iyy="1e-6" iyz="0" izz="1e-6"/>
+        </inertial>
+        <collision name='camera_collision'>
+            <origin xyz="0.0 0 0" rpy=" 0 0 0"/>
+            <geometry>
+                <box size=".05 .05 .05"/>
+            </geometry>
+        </collision>
+        <visual name='camera_visual'>
+            <origin xyz="0.0 0 0" rpy=" 0 0 0"/>
+            <geometry>
+                <box size=".05 .05 .05"/>
+            </geometry>
+        </visual>
+    </link>
+    <joint type="fixed" name="camera_joint">
+        <origin xyz="0.4 0 0" rpy="0 0 0"/>
+        <child link="camera"/>
+        <parent link="chassis"/>
+    </joint>
+    <link name='hokuyo'>
+        <inertial>
+            <mass value="0.1"/>
+            <origin xyz="0.0 0 0" rpy=" 0 0 0"/>
+            <inertia ixx="1e-6" ixy="0" ixz="0" iyy="1e-6" iyz="0" izz="1e-6"/>
+        </inertial>
+        <collision name='hokuyo_collision'>
+            <origin xyz="0.0 0 0" rpy=" 0 0 0"/>
+            <geometry>
+                <box size=".1 .1 .1"/>
+            </geometry>
+        </collision>
+        <visual name='hokuyo_visual'>
+            <origin xyz="0.0 0 0" rpy=" 0 0 0"/>
+            <geometry>
+                <mesh filename="package://roborock/meshes/hokuyo.dae"/>
+            </geometry>
+        </visual>
+    </link>
+    <joint type="fixed" name="hokuyo_joint">
+        <origin xyz="-0.2 0 .1" rpy="0 0 0"/>
+        <child link="hokuyo"/>
+        <parent link="chassis"/>
+    </joint>
 </robot>

Commit message: add color tag for casters

File: roborock/urdf/roborock.xacro (robot description, xacro)
@@ -7,4 +7,7 @@
     <material name="black">
         <color rgba="0 0 0 1"/>
+    </material>
+    <material name="slightly_yellow">
+        <color rgba="255 255 204 1"/>
     </material>
     <link name="robot_footprint"></link>
@@ -45,4 +48,5 @@
                 <sphere radius="0.05"/>
             </geometry>
+            <material name="slightly_yellow"/>
         </visual>
         <collision name='front_caster_collision'>
@@ -57,4 +61,5 @@
                 <sphere radius="0.05"/>
             </geometry>
+            <material name="slightly_yellow"/>
         </visual>
     </link>
