Commit message: adjust the model

File: roborock/urdf/roborock.xacro (robot description, xacro)
@@ -27,5 +27,5 @@
             <origin xyz="0 0 0" rpy=" 0 0 0"/>
             <geometry>
-                <cylinder radius="0.4" length="0.15"/>
+                <cylinder radius="0.3" length="0.15"/>
             </geometry>
         </collision>
@@ -65,5 +65,5 @@
     </link>
     <joint type="continuous" name="left_wheel_hinge">
-        <origin xyz="0 0.25 -0.025" rpy="0 0 0"/>
+        <origin xyz="0 0.23 -0.025" rpy="0 0 0"/>
         <child link="left_wheel"/>
         <parent link="chassis"/>
@@ -93,5 +93,5 @@
     </link>
     <joint type="continuous" name="right_wheel_hinge">
-        <origin xyz="0 -0.25 -0.025" rpy="0 0 0"/>
+        <origin xyz="0 -0.23 -0.025" rpy="0 0 0"/>
         <child link="right_wheel"/>
         <parent link="chassis"/>
@@ -164,5 +164,5 @@
     </link>
     <joint type="fixed" name="hokuyo_joint">
-        <origin xyz="-0.2 0 .1" rpy="0 0 0"/>
+        <origin xyz="0 0 .1" rpy="0 0 0"/>
         <child link="hokuyo"/>
         <parent link="chassis"/>

Commit message: change color

File: roborock/urdf/roborock.xacro (robot description, xacro)
@@ -2,6 +2,6 @@
 <robot name="roborock" xmlns:xacro="http://www.ros.org/wiki/xacro">
     <xacro:include filename="$(find roborock)/urdf/roborock.gazebo"/>
-    <material name="army_green">
-        <color rgba="51 153 102 1"/>
+    <material name="light_blue">
+        <color rgba="0 170 255 1"/>
     </material>
     <material name="black">
@@ -35,5 +35,5 @@
                 <cylinder radius="0.4" length="0.15"/>
             </geometry>
-            <material name="army_green"/>
+            <material name="light_blue"/>
         </visual>
         <collision name='back_caster_collision'>

Commit message: make it smaller

File: roborock/urdf/roborock.xacro (robot description, xacro)
@@ -33,5 +33,5 @@
             <origin xyz="0 0 0" rpy=" 0 0 0"/>
             <geometry>
-                <cylinder radius="0.4" length="0.15"/>
+                <cylinder radius="0.3" length="0.15"/>
             </geometry>
             <material name="light_blue"/>

Commit message: fine tune the model

File: roborock/urdf/roborock.xacro (robot description, xacro)
@@ -44,5 +44,5 @@
         </collision>
         <visual name='back_caster_visual'>
-            <origin xyz="-0.25 0 -0.075" rpy=" 0 0 0"/>
+            <origin xyz="-0.23 0 -0.075" rpy=" 0 0 0"/>
             <geometry>
                 <sphere radius="0.05"/>
@@ -51,5 +51,5 @@
         </visual>
         <collision name='front_caster_collision'>
-            <origin xyz="0.25 0 -0.075" rpy=" 0 0 0"/>
+            <origin xyz="0.23 0 -0.075" rpy=" 0 0 0"/>
             <geometry>
                 <sphere radius="0.0499"/>
@@ -140,5 +140,5 @@
     </link>
     <joint type="fixed" name="camera_joint">
-        <origin xyz="0.4 0 0" rpy="0 0 0"/>
+        <origin xyz="0.3 0 0" rpy="0 0 0"/>
         <child link="camera"/>
         <parent link="chassis"/>

Commit message: two more tags to change

File: roborock/urdf/roborock.xacro (robot description, xacro)
@@ -38,5 +38,5 @@
         </visual>
         <collision name='back_caster_collision'>
-            <origin xyz="-0.25 0 -0.075" rpy=" 0 0 0"/>
+            <origin xyz="-0.23 0 -0.075" rpy=" 0 0 0"/>
             <geometry>
                 <sphere radius="0.0499"/>
@@ -57,5 +57,5 @@
         </collision>
         <visual name='front_caster_visual'>
-            <origin xyz="0.25 0 -0.075" rpy=" 0 0 0"/>
+            <origin xyz="0.23 0 -0.075" rpy=" 0 0 0"/>
             <geometry>
                 <sphere radius="0.05"/>

Commit message: adjust model

File: roborock/urdf/roborock.xacro (robot description, xacro)
@@ -27,5 +27,5 @@
             <origin xyz="0 0 0" rpy=" 0 0 0"/>
             <geometry>
-                <cylinder radius="0.3" length="0.15"/>
+                <cylinder radius="0.2" length="0.15"/>
             </geometry>
         </collision>
@@ -33,10 +33,10 @@
             <origin xyz="0 0 0" rpy=" 0 0 0"/>
             <geometry>
-                <cylinder radius="0.3" length="0.15"/>
+                <cylinder radius="0.2" length="0.15"/>
             </geometry>
             <material name="light_blue"/>
         </visual>
         <collision name='back_caster_collision'>
-            <origin xyz="-0.23 0 -0.075" rpy=" 0 0 0"/>
+            <origin xyz="-0.13 0 -0.075" rpy=" 0 0 0"/>
             <geometry>
                 <sphere radius="0.0499"/>
@@ -44,5 +44,5 @@
         </collision>
         <visual name='back_caster_visual'>
-            <origin xyz="-0.23 0 -0.075" rpy=" 0 0 0"/>
+            <origin xyz="-0.13 0 -0.075" rpy=" 0 0 0"/>
             <geometry>
                 <sphere radius="0.05"/>
@@ -51,5 +51,5 @@
         </visual>
         <collision name='front_caster_collision'>
-            <origin xyz="0.23 0 -0.075" rpy=" 0 0 0"/>
+            <origin xyz="0.13 0 -0.075" rpy=" 0 0 0"/>
             <geometry>
                 <sphere radius="0.0499"/>
@@ -57,5 +57,5 @@
         </collision>
         <visual name='front_caster_visual'>
-            <origin xyz="0.23 0 -0.075" rpy=" 0 0 0"/>
+            <origin xyz="0.13 0 -0.075" rpy=" 0 0 0"/>
             <geometry>
                 <sphere radius="0.05"/>
@@ -65,5 +65,5 @@
     </link>
     <joint type="continuous" name="left_wheel_hinge">
-        <origin xyz="0 0.23 -0.025" rpy="0 0 0"/>
+        <origin xyz="0 0.13 -0.025" rpy="0 0 0"/>
         <child link="left_wheel"/>
         <parent link="chassis"/>
@@ -93,5 +93,5 @@
     </link>
     <joint type="continuous" name="right_wheel_hinge">
-        <origin xyz="0 -0.23 -0.025" rpy="0 0 0"/>
+        <origin xyz="0 -0.13 -0.025" rpy="0 0 0"/>
         <child link="right_wheel"/>
         <parent link="chassis"/>
@@ -140,5 +140,5 @@
     </link>
     <joint type="fixed" name="camera_joint">
-        <origin xyz="0.3 0 0" rpy="0 0 0"/>
+        <origin xyz="0.21 0 0" rpy="0 0 0"/>
         <child link="camera"/>
         <parent link="chassis"/>
@@ -164,5 +164,5 @@
     </link>
     <joint type="fixed" name="hokuyo_joint">
-        <origin xyz="0 0 .1" rpy="0 0 0"/>
+        <origin xyz="0 0 .2" rpy="0 0 0"/>
         <child link="hokuyo"/>
         <parent link="chassis"/>

Commit message: adjust model

File: roborock/urdf/roborock.xacro (robot description, xacro)
@@ -27,5 +27,5 @@
             <origin xyz="0 0 0" rpy=" 0 0 0"/>
             <geometry>
-                <cylinder radius="0.3" length="0.15"/>
+                <cylinder radius="0.2" length="0.15"/>
             </geometry>
         </collision>
@@ -33,10 +33,10 @@
             <origin xyz="0 0 0" rpy=" 0 0 0"/>
             <geometry>
-                <cylinder radius="0.3" length="0.15"/>
+                <cylinder radius="0.2" length="0.15"/>
             </geometry>
             <material name="light_blue"/>
         </visual>
         <collision name='back_caster_collision'>
-            <origin xyz="-0.23 0 -0.075" rpy=" 0 0 0"/>
+            <origin xyz="-0.18 0 -0.075" rpy=" 0 0 0"/>
             <geometry>
                 <sphere radius="0.0499"/>
@@ -44,5 +44,5 @@
         </collision>
         <visual name='back_caster_visual'>
-            <origin xyz="-0.23 0 -0.075" rpy=" 0 0 0"/>
+            <origin xyz="-0.18 0 -0.075" rpy=" 0 0 0"/>
             <geometry>
                 <sphere radius="0.05"/>
@@ -51,5 +51,5 @@
         </visual>
         <collision name='front_caster_collision'>
-            <origin xyz="0.23 0 -0.075" rpy=" 0 0 0"/>
+            <origin xyz="0.18 0 -0.075" rpy=" 0 0 0"/>
             <geometry>
                 <sphere radius="0.0499"/>
@@ -57,5 +57,5 @@
         </collision>
         <visual name='front_caster_visual'>
-            <origin xyz="0.23 0 -0.075" rpy=" 0 0 0"/>
+            <origin xyz="0.18 0 -0.075" rpy=" 0 0 0"/>
             <geometry>
                 <sphere radius="0.05"/>
@@ -65,5 +65,5 @@
     </link>
     <joint type="continuous" name="left_wheel_hinge">
-        <origin xyz="0 0.23 -0.025" rpy="0 0 0"/>
+        <origin xyz="0 0.18 -0.025" rpy="0 0 0"/>
         <child link="left_wheel"/>
         <parent link="chassis"/>
@@ -93,5 +93,5 @@
     </link>
     <joint type="continuous" name="right_wheel_hinge">
-        <origin xyz="0 -0.23 -0.025" rpy="0 0 0"/>
+        <origin xyz="0 -0.18 -0.025" rpy="0 0 0"/>
         <child link="right_wheel"/>
         <parent link="chassis"/>
@@ -140,5 +140,5 @@
     </link>
     <joint type="fixed" name="camera_joint">
-        <origin xyz="0.3 0 0" rpy="0 0 0"/>
+        <origin xyz="0.21 0 0" rpy="0 0 0"/>
         <child link="camera"/>
         <parent link="chassis"/>
@@ -164,5 +164,5 @@
     </link>
     <joint type="fixed" name="hokuyo_joint">
-        <origin xyz="0 0 .1" rpy="0 0 0"/>
+        <origin xyz="0 0 .2" rpy="0 0 0"/>
         <child link="hokuyo"/>
         <parent link="chassis"/>

Commit message: adjust model

File: roborock/urdf/roborock.xacro (robot description, xacro)
@@ -164,5 +164,5 @@
     </link>
     <joint type="fixed" name="hokuyo_joint">
-        <origin xyz="0 0 .2" rpy="0 0 0"/>
+        <origin xyz="0 0 .1" rpy="0 0 0"/>
         <child link="hokuyo"/>
         <parent link="chassis"/>
